File: mini-ten-key-plus.kicad_pcb (KiCad board)
At the start: 2 copper layers, 45 parts, among them SW0 SW_Push, U0 ProMicro

Commit message: Did practice col/row wiring
Parts:
- moved SW0 15.6 mm to (81.0, 41.3), turned to 270 degrees
- moved D19 10.3 mm to (73.0, 107.2)
- moved D18 2.38 mm to (73.0, 109.5)
Connections:
- U0 pad 10: Net-(U0-Pad10) -> IO
- U0 pad 11: Net-(U0-Pad11) -> IO
- U0 pad 12: Net-(U0-Pad12) -> IO
- U0 pad 17: Net-(U0-Pad17) -> IO
- U0 pad 18: Net-(U0-Pad18) -> IO
- U0 pad 19: Net-(U0-Pad19) -> IO
- U0 pad 20: Net-(U0-Pad20) -> IO
- U0 pad 7: Net-(U0-Pad7) -> IO
- U0 pad 8: Net-(U0-Pad8) -> IO
- U0 pad 9: Net-(U0-Pad9) -> IO
Routing:
- net IO: track 0.00 -> 235.4 mm
- net RESET: track 7.13 -> 28.1 mm
- net GND: track 37.5 -> 53.1 mm
- net Net-(D19-Pad2): track 11.9 -> 23.0 mm
- net ROW4: track 54.8 -> 44.2 mm
- net COL3: track 93.3 -> 90.4 mm
- net Net-(D18-Pad2): track 6.46 -> 4.13 mm
